File: source/aREF2048.sch (KiCad schematic (older format))
At the start: 34 parts, among them J1 BATT, J2 VREF, J3 GND, Q1 IRLML6401, U1 TPS3809K33, U2 LTC6655CHMS8-2.048, U3 LTC2054, U4 OPA365

Commit message: Version 0.1
Parts:
- added F1: 200mA, Fuse:Fuse_0805_2012Metric_Pad1.15x1.40mm_HandSolder, symbol Device:Polyfuse
- H1, H2, H3, H4: footprint MountingHole:MountingHole_2.7mm_M2.5_Pad -> MountingHole:MountingHole_2.2mm_M2
- Q1, U1: footprint Package_TO_SOT_SMD:SOT-23_Handsoldering -> Package_TO_SOT_SMD:SOT-23
- U3, U4: footprint Package_TO_SOT_SMD:SOT-23-5_HandSoldering -> Package_TO_SOT_SMD:SOT-23-5
Connections:
- net at Q1.3 (D): now also F1.1; no longer J1.1 (Pin_1)
- new net: F1.2, J1.1 (Pin_1)
Other:
- moved on the sheet: C5, C7, D1, H1, H2, H3, H4, J1, R1, U1
